File: kiCad/kiCad.kicad_sch (KiCad schematic)
At the start: 0 parts

Commit message: erster commit
Parts:
- added D1: 1N4007, Diode_THT:D_DO-41_SOD81_P10.16mm_Horizontal, symbol Diode:1N4007
- added Lock: ~, symbol Device:L
- added Q1: IRLZ34N, Package_TO_SOT_THT:TO-220-3_Vertical, symbol Transistor_FET:IRLZ34N
- added R1: 10 K, symbol Device:R
- added R2: 330, symbol Device:R
- added U1: ESP32-WROOM-32, RF_Module:ESP32-WROOM-32, symbol RF_Module:ESP32-WROOM-32
Connections:
- new net: R2.1, U1.14 (IO12)
- new net: Q1.1 (G), R1.1, R2.2
- new net: D1.2 (A), Lock.1, Q1.2 (D)
- new net +12V: D1.1 (K), Lock.2
- new net +5V: U1.2 (VDD)
- new net Earth: Q1.3 (S), R1.2, U1.1 (GND), U1.15 (GND), U1.38 (GND), U1.39 (GND)
